File: keyboard/PCB/PCB.kicad_sch (KiCad schematic)
At the start: 83 parts, among them U1 Arduino_Pro_Micro

Commit message: Updated
Parts:
- removed D1, D10, D11, D12, D13, D14, D15, D16, D17, D18, D19, D2, D20, D21, D22, D23, D24, D25, D26, D27, D28, D29, D3, D30, D31, D32, D33, D34, D35, D36, D37, D38, D39, D4, D40, D41, D5, D6, D7, D8, D9: (no value), symbol ScottoKeebs:Placeholder_Diode
- removed S1, S10, S11, S12, S13, S14, S15, S16, S17, S18, S19, S2, S20, S21, S22, S23, S24, S25, S26, S27, S28, S29, S3, S30, S31, S32, S33, S34, S35, S36, S37, S38, S39, S4, S40, S41, S5, S6, S7, S8, S9: (no value), symbol ScottoKeebs:Placeholder_Keyswitch
- removed U1: Arduino_Pro_Micro, ScottoKeebs_MCU:Arduino_Pro_Micro, symbol ScottoKeebs:MCU_Arduino_Pro_Micro
- added J3: OLED_128x64, ScottoKeebs_Components:OLED_128x64, symbol ScottoKeebs:OLED_128x64
- added U1: STM32F411CEUx, Package_DFN_QFN:QFN-48-1EP_7x7mm_P0.5mm_EP5.6x5.6mm, symbol MCU_ST_STM32F4:STM32F411CEUx
- added U2: Arduino_Pro_Micro, ScottoKeebs_MCU:Arduino_Pro_Micro, symbol ScottoKeebs:MCU_Arduino_Pro_Micro
- added U3: TRRS, ScottoKeebs_Components:TRRS_PJ-320A, symbol ScottoKeebs:Placeholder_TRRS
Connections:
- net C0: now also U1.10 (PA0), U2.7 (4/PD4)
- net C1: now also U1.11 (PA1), U2.8 (5/PC6)
- net C2: now also U1.18 (PB0), U2.9 (6/PD7)
- net C3: now also U1.19 (PB1), U2.10 (7/PE6)
- net C4: now also U1.14 (PA4), U2.11 (8/PB4)
- net C5: now also U1.15 (PA5), U2.12 (9/PB5)
- net C6: now also U1.16 (PA6), U2.13 (10/PB6)
- net C7: now also U1.17 (PA7), U2.15 (14/PB3)
- net R0: now also U1.21 (PB10), U2.16 (15/PB1)
- net R1: now also U1.25 (PB12), U2.14 (16/PB2)
- net R2: now also U1.26 (PB13), U2.17 (A0/PF7)
- net R3: now also U1.27 (PB14), U2.18 (A1/PF6)
- net R4: now also U1.28 (PB15), U2.19 (A2/PF5)
- new net +3V3: U1.1 (VBAT), U1.24 (VDD), U1.36 (VDD), U1.48 (VDD), U1.9 (VDDA)
- new net BOOT: U1.20 (PB2), U1.44 (BOOT0)
- new net D+: U1.33 (PA12)
- new net D-: U1.32 (PA11)
- new net Flashing: U1.34 (PA13), U1.37 (PA14)
- new net GND: J3.1 (GND), U1.23 (VSS), U1.35 (VSS), U1.47 (VSS), U1.49 (VSS), U1.8 (VSSA), U2.23 (GND), U2.3 (GND), U2.4 (GND), U3.4 (RING2)
- new net RX: U1.13 (PA3), U2.2 (RX1/PD2), U3.3 (RING1)
- new net SCL: J3.3 (SCL), U1.42 (PB6), U2.6 (3/PD0)
- new net SDA: J3.4 (SDA), U1.43 (PB7), U2.5 (2/PD1)
- new net TX: U1.12 (PA2), U2.1 (TX0/PD3), U3.2 (TIP)
- new net VCC: J3.2 (VCC), U2.21 (VCC), U3.1 (SLEEVE)
Other:
- added sheet extras (extras.kicad_sch)
- added sheet key_matrix (key_matrix.kicad_sch)
- added sheet power (power.kicad_sch)
