File: Macropad/Macropad_v2/PCB/.history/PCB.kicad_pcb (KiCad board)
At the start: 2 copper layers, 139 x 123.8 mm, 106 parts, among them J1 USB_C_Receptacle_USB2.0_14P, J2 OLED_128x64, J3 Micro_SD_Card_Det1, SW1 SW_Push, SW2 RotaryEncoder, SW3 RotaryEncoder, U1 STM32F072CBTx, U2 USBLC6-2SC6, U3 XC6206, U5 TRRS

Commit message: Updated
Parts:
- removed the C10 at (235.5, 87.1)
- removed the C11 at (235.5, 90.1)
- removed the C12 at (235.5, 93.1)
- removed the C13 at (235.5, 96.2)
- removed J3: Micro_SD_Card_Det1, Connector_Card:microSD_HC_Hirose_DM3AT-SF-PEJM5
- removed the R10 at (226.7, 87.1)
- removed the R11 at (226.7, 90.0)
- removed the R12 at (226.7, 93.0)
- removed R13, R14, R16, R17: 10k, Resistor_SMD:R_0805_2012Metric
- removed the R15 at (231.1, 90.0)
- removed the R4 at (222.3, 87.1)
- removed the R5 at (222.3, 90.0)
- removed the R6 at (222.3, 93.0)
- removed the R7 at (222.3, 95.9)
- removed the SW2 at (203.5, 67.4)
- removed the SW3 at (203.5, 83.1)
Connections:
- U1 pad 12: SLIDER_2 -> unconnected-(U1-PA2-Pad12)
- U1 pad 13: SLIDER_1 -> unconnected-(U1-PA3-Pad13)
- U1 pad 14: CS -> unconnected-(U1-PA4-Pad14)
- U1 pad 15: IS_SD -> unconnected-(U1-PA5-Pad15)
- U1 pad 26: SCK -> unconnected-(U1-PB13-Pad26)
- U1 pad 27: MISO -> SLIDER_1
- U1 pad 28: MOSI -> SLIDER_2
Routing:
- net GND: track 509.8 -> 508.6 mm
