File: Macropad/PCB/.history/PCB.kicad_pcb (KiCad board)
At the start: 2 copper layers, 139 x 123.8 mm, 106 parts, among them J1 USB_C_Receptacle_USB2.0_14P, J2 OLED_128x64, J3 Micro_SD_Card_Det1, SW1 SW_Push, SW2 RotaryEncoder, SW3 RotaryEncoder, U1 STM32F072CBTx, U2 USBLC6-2SC6, U3 XC6206, U5 TRRS

Commit message: Updated macropad
Parts:
- removed the SW2 at (32.2, 43.5)
- removed the SW3 at (50.0, 44.0)
- moved SW2 172.9 mm to (32.2, 43.5)
- moved SW3 158.6 mm to (50.0, 43.5)
- moved J3 40.6 mm to (195.5, 47.5), turned to 180 degrees
- moved R7 1.09 mm to (54.5, 33.5)
- moved R10 1.04 mm to (59.0, 33.5)
- moved C10 1.00 mm to (57.0, 36.5)
- moved R6 1.00 mm to (51.0, 33.5)
- moved R11 0.59 mm to (64.5, 34.0)
Routing:
- net +3.3V: track 338.5 -> 343.9 mm
- net Net-(R11-Pad1): track 27.2 -> 24.5 mm
- net Net-(R10-Pad1): track 34.4 -> 36.4 mm
- net GND: track 509.8 -> 511.5 mm
- net RE_2_B: track 41.3 -> 42.5 mm
