File: Macropad/PCB/.history/PCB.kicad_sch (KiCad schematic)
At the start: 46 parts, among them J1 USB_C_Receptacle_USB2.0_14P, J2 OLED_128x64, J3 Micro_SD_Card_Det1, SW1 SW_Push, SW2 RotaryEncoder, SW3 RotaryEncoder, U1 STM32F072CBTx, U2 USBLC6-2SC6, U3 XC6206, U5 TRRS

Commit message: Updated
Parts:
- added C14, C15: 10nF, symbol Device:C
- added R18, R19: 100, symbol Device:R
- added RV1, RV2: 10k, symbol Device:R_Potentiometer
Connections:
- net +3.3V: now also RV1.3, RV2.1
- net GND: now also C14.1, C15.2, RV1.1, RV2.3
- new net: R19.1, RV2.2
- new net: R18.2, RV1.2
- new net ADC_X: C14.2, R18.1
- new net ADC_Y: C15.1, R19.2
- no-connect marks 0 -> 1
